File: Hardware/ETHERNET_PHY.kicad_sch (KiCad schematic)
At the start: 20 parts, among them J13 RJ45_Hanrun_HR911105A_Horizon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, U39 JL1111-N032I

Commit message: 拉线
Parts:
- renumbered C101 to C102, C108 to C109, C115 to C125, C118 to C128, C119 to C129, C120 to C130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

Commit message: 修存档拉线
Parts:
- renumbered C102 to C89, C125 to C90, C128 to C91, C129 to C92, C130 to C93, C89 to C94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
