File: Hardware/INVERTER_BRIDGE.kicad_sch (KiCad schematic)
At the start: 68 parts, among them Q1 CSD19532Q5B, Q2 CSD19532Q5B, Q3 CSD19532Q5B, Q4 CSD19532Q5B, Q5 CSD19532Q5B, Q6 CSD19532Q5B, U10 UCC27282DRCR, U11 INA240A1PWR, U12 UCC27282DRCR, U13 INA240A1PWR, U14 UCC27282DRCR, U15 INA240A1PWR, U16 INA240A1PWR

Commit message: 拉线
Parts:
- removed R40: 10K,1%, Resistor_SMD:R_0402_1005Metric, symbol HPM6280Foc:0402WGF1002TCE
- added U51: 74LVC1G08, Package_TO_SOT_SMD:SOT-353_SC-70-5, symbol 74xGxx:74LVC1G08
- renumbered C50 to C67, C51 to C68, C52 to C69, C53 to C70, C54 to C71, C55 to C72, C56 to C73, C57 to C74, C58 to C75, C59 to C76, C60 to C77, C61 to C78, C62 to C79, C63 to C80, C64 to C81, C65 to C82, C66 to C83, D6 to D15, D7 to D16, D8 to D17, D9 to D18, D10 to D19, D11 to D20, D12 to D21, D13 to D22, D14 to D23, J7 to J10, J5 to J8, J6 to J9, NT4 to NT10, NT5 to NT11, NT6 to NT12, NT17 to NT19, NT18 to NT20, NT1 to NT7, NT2 to NT8, NT3 to NT9, Q4 to Q10, Q5 to Q11, Q6 to Q12, Q1 to Q7, Q2 to Q8, Q3 to Q9, R23 to R41, R24 to R42, R25 to R43, R26 to R44, R27 to R45, R28 to R46, R29 to R47, R30 to R48, R31 to R49, R32 to R50, R33 to R51, R34 to R52, R35 to R53, R36 to R54, R37 to R55, R38 to R56, R39 to R57, U10 to U17, U11 to U18, U12 to U19, U13 to U20, U14 to U21, U15 to U22, U16 to U23
Connections:
- net DRIVER.EN: now also U51.1; no longer U17.6 (EN), U19.6 (EN), U21.6 (EN)
- new net +3.3V: U51.5 (VCC)
- new net BREAK: U51.2
- new net EN: U17.6 (EN), U19.6 (EN), U21.6 (EN), U51.4
- new net GND: U51.3 (GND)

Commit message: 修存档拉线
Parts:
- renumbered C67 to C31, C68 to C32, C69 to C33, C70 to C34, C71 to C35, C72 to C36, C73 to C37, C74 to C38, C75 to C39, C76 to C40, C77 to C41, C78 to C42, C79 to C43, C80 to C44, C81 to C45, C82 to C46, C83 to C47, D15 to D14, D16 to D15, D17 to D16, D18 to D17, D19 to D18, D20 to D19, D21 to D20, D22 to D21, D23 to D22, J8 to J7, J9 to J8, J10 to J9, NT7 to NT1, NT8 to NT2, NT9 to NT3, NT10 to NT4, NT11 to NT5, NT12 to NT6, NT19 to NT7, NT20 to NT8, Q7 to Q1, Q8 to Q2, Q9 to Q3, Q10 to Q4, Q11 to Q5, Q12 to Q6, R41 to R27, R42 to R28, R43 to R29, R44 to R30, R45 to R31, R46 to R32, R47 to R33, R48 to R34, R49 to R35, R50 to R36, R51 to R37, R52 to R38, R53 to R39, R54 to R40, R55 to R41, R56 to R42, R57 to R43, U17 to U12, U18 to U13, U19 to U14, U20 to U15, U21 to U16, U22 to U17, U51 to U18, U23 to U19

Commit message: 拉线
Other:
- note added: "硬件STO"
Changed lines of the file:
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@@
 	(generator_version "9.0")
 	(paper "A4")
+	(text "硬件STO"
+		(exclude_from_sim no)
+		(at 29.718 166.878 0)
+		(effects
+			(font
+				(size 1.27 1.27)
+			)
+		)
+	)
 	(junction
 		(at 148.59 177.8)
@@
 			)
 			(justify left)
+		)
+	)
+	(rule_area
+		(polyline
+			(pts
+				(xy 13.97 64.77) (xy 140.97 64.77) (xy 140.97 19.05) (xy 13.97 19.05)
+			)
+			(stroke
+				(width 0)
+				(type dash)
+			)
+			(fill
+				(type none)
+			)
+		)
+	)
+	(rule_area
+		(polyline
+			(pts
+				(xy 13.97 111.76) (xy 140.97 111.76) (xy 140.97 66.04) (xy 13.97 66.04)
+			)
+			(stroke
+				(width 0)
+				(type dash)
+			)
+			(fill
+				(type none)
+			)
 		)
 	)
@@
 			)
 			(stroke
-				(width 0)
-				(type dash)
-			)
-			(fill
-				(type none)
-			)
-		)
-	)
-	(rule_area
-		(polyline
-			(pts
-				(xy 13.97 111.76) (xy 140.97 111.76) (xy 140.97 66.04) (xy 13.97 66.04)
-			)
-			(stroke
-				(width 0)
-				(type dash)
-			)
-			(fill
-				(type none)
-			)
-		)
-	)
-	(rule_area
-		(polyline
-			(pts
-				(xy 13.97 64.77) (xy 140.97 64.77) (xy 140.97 19.05) (xy 13.97 19.05)
-			)
-			(stroke

Commit message: 拉线
Parts:
- added C152: 100nF,16V, Capacitor_SMD:C_0402_1005Metric, symbol HPM6280Foc:CC0402KRX7R7BB104
Connections:
- net GND: now also C152.1
- net +3.3V renamed +3.3_2
- net +3.3_2: now also C152.2
Changed lines of the file:
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@@
 	)
 	(junction
+		(at 48.26 166.37)
+		(diameter 0)
+		(color 0 0 0 0)
+	)
+	(junction
 		(at 92.71 40.64)
 		(diameter 0)
@@
 	)
 	(symbol
+		(lib_id "power:GND")
+		(at 58.42 166.37 90)
+		(unit 1)
+		(exclude_from_sim no)
+		(in_bom yes)
+		(on_board yes)
+		(dnp no)
+		(fields_autoplaced yes)
+		(property "Reference" "#PWR0345"
+			(at 64.77 166.37 0)
+			(effects
+				(font
+					(size 1.27 1.27)
+				)
+				(hide yes)
+			)
+		)
+		(property "Value" "GND"
+			(at 62.23 166.3699 90)
+			(effects
+				(font
+					(size 1.27 1.27)
+				)
+				(justify right)
+			)
+		)
+		(property "Footprint" ""
+			(at 58.42 166.37 0)
+			(effects
+				(font
+					(size 1.27 1.27)
+				)
+				(hide yes)
+			)
+		)
+		(property "Datasheet" ""
+			(at 58.42 166.37 0)
+			(effects
+				(font
+					(size 1.27 1.27)
+				)
+				(hide yes)
+			)
+		)
+		(property "Description" "Power symbol creates a global label with name \"GND\" , ground"
+			(at 58.42 166.37 0)
+			(effects
+				(font
+					(size 1.27 1.27)
+				)
+				(hide yes)
+			)
+		)
+		(pin "1"
+		)
+		(instances
+			(project "HPM5E31_ECatDualFOC"
+				(path "/a07e9810-3899-4327-ba8f-f24142a7c70e/0dcd211e-0cd3-4a5b-8381-64e2d1ceb9a5"
+					(reference "#PWR0345")
+					(unit 1)
+				)
+				(path "/a07e9810-3899-4327-ba8f-f24142a7c70e/395dcadf-6728-482a-9c72-95a7205ca2d1"
+					(reference "#PWR0348")
+					(unit 1)
+				)
+			)
+		)
+	)
+	(symbol
 		(lib_id "HPM6280Foc:CL31B105KCHNNNE")
 		(at 109.22 82.55 180)
@@
 	)
 	(symbol
+		(lib_id "HPM6280Foc:+3.3_2")
+		(at 48.26 165.1 180)
+		(unit 1)
+		(exclude_from_sim no)
+		(in_bom yes)
+		(on_board yes)
+		(dnp no)
+		(property "Reference" "#PWR0121"
+			(at 49.53 162.56 0)
+			(effects
+				(font
+					(size 1.27 1.27)
+				)
+				(hide yes)
+			)
+		)
+		(property "Value" "+3.3_2"
+			(at 47.498 162.306 0)
+			(effects
+				(font
+					(size 1.27 1.27)
+				)
+			)
+		)
+		(property "Footprint" ""
+			(at 48.26 165.1 0)
+			(effects
+				(font
+					(size 1.27 1.27)
+				)
+				(hide yes)
+			)
+		)
+		(property "Datasheet" ""
+			(at 48.26 165.1 0)
+			(effects
+				(font
+					(size 1.27 1.27)
+				)
+				(hide yes)
+			)
+		)
+		(property "Description" "电源符号创建名为 '+3.3_2' 的全局标签"
+			(at 48.26 165.1 0)
+			(effects
+				(font
+					(size 1.27 1.27)
+				)
+				(hide yes)
+			)
+		)
+		(pin ""
+		)
+		(instances
+			(project ""
+				(path "/a07e9810-3899-4327-ba8f-f24142a7c70e/0dcd211e-0cd3-4a5b-8381-64e2d1ceb9a5"
+					(reference "#PWR0121")
+					(unit 1)
+				)
+				(path "/a07e9810-3899-4327-ba8f-f24142a7c70e/395dcadf-6728-482a-9c72-95a7205ca2d1"
+					(reference "#PWR0162")
+					(unit 1)
+				)
+			)
+		)
+	)
+	(symbol
 		(lib_id "HPM6280Foc:CSD19532Q5B")
 		(at 100.33 101.6 0)
@@
 	)
 	(symbol
-		(lib_id "power:+3.3V")
-		(at 48.26 166.37 0)
-		(unit 1)
-		(exclude_from_sim no)
-		(in_bom yes)
-		(on_board yes)
-		(dnp no)
-		(fields_autoplaced yes)
-		(property "Reference" "#PWR0121"
-			(at 48.26 170.18 0)
-			(effects
-				(font
-					(size 1.27 1.27)
-				)
-				(hide yes)
-			)
-		)
-		(property "Value" "+3.3V"
-			(at 48.26 161.29 0)
-			(effects
-				(font
-					(size 1.27 1.27)
-				)
-			)
-		)
-		(property "Footprint" ""
-			(at 48.26 166.37 0)
-			(effects
-				(font
-					(size 1.27 1.27)
-				)
-				(hide yes)
-			)
-		)
-		(property "Datasheet" ""
-			(at 48.26 166.37 0)
-			(effects
-				(font
-					(size 1.27 1.27)
-				)
-				(hide yes)
-			)
-		)
-		(property "Description" "Power symbol creates a global label with name \"+3.3V\""
-			(at 48.26 166.37 0)
-			(effects
-				(font
-					(size 1.27 1.27)
-				)
-				(hide yes)
-			)
-		)
-		(pin "1"
-		)
-		(instances
-			(project "HPM5E31_ECatDualFOC"
-				(path "/a07e9810-3899-4327-ba8f-f24142a7c70e/0dcd211e-0cd3-4a5b-8381-64e2d1ceb9a5"
-					(reference "#PWR0121")
-					(unit 1)
-				)
-				(path "/a07e9810-3899-4327-ba8f-f24142a7c70e/395dcadf-6728-482a-9c72-95a7205ca2d1"
-					(reference "#PWR0162")
-					(unit 1)
-				)
-			)
-		)
-	)
-	(symbol
 		(lib_id "Device:NetTie_2")
 		(at 133.35 50.8 0)
@@
 					(unit 1)
 				)
+			)
+		)
+	)
+	(symbol
+		(lib_id "HPM6280Foc:CC0402KRX7R7BB104")
+		(at 53.34 166.37 0)
+		(unit 1)
+		(exclude_from_sim no)
+		(in_bom yes)
+		(on_board yes)
+		(dnp no)
+		(property "Reference" "C152"
+			(at 57.658 164.592 0)
+			(effects
+				(font
+					(size 1.27 1.27)
+				)
+			)
+		)
+		(property "Value" "100nF,16V"
+			(at 56.134 162.56 0)
+			(effects
+				(font
+					(size 1.27 1.27)
+				)
+			)
+		)
+		(property "Footprint" "Capacitor_SMD:C_0402_1005Metric"
+			(at 53.34 166.37 0)
+			(effects
+				(font
+					(size 1.27 1.27)
+				)
+				(hide yes)
+			)
+		)
+		(property "Datasheet" ""
+			(at 53.34 166.37 0)
+			(effects
+				(font
+					(size 1.27 1.27)
+				)
+				(hide yes)
+			)
+		)
+		(property "Description" ""
+			(at 53.34 166.37 0)
+			(effects
+				(font
+					(size 1.27 1.27)
+				)
+				(hide yes)
+			)
+		)
+		(property "制造商编号" ""
+			(at 53.34 166.37 0)
+			(effects
+				(font
+					(size 1.27 1.27)
+				)
+				(hide yes)
+			)
+		)
+		(property "制造商" "YAGEO(国巨)"
+			(at 53.34 166.37 0)
+			(effects
+				(font
+					(size 1.27 1.27)
+				)
+				(hide yes)
+			)
+		)
+		(property "华秋编号" "G0042289"
+			(at 53.34 166.37 0)
+			(effects
+				(font
+					(size 1.27 1.27)
+				)
+				(hide yes)
+			)
+		)
+		(property "立创编号" "C60474"
+			(at 49.53 170.18 0)
+			(effects
+				(font
+					(size 1.27 1.27)
+				)
+				(hide yes)
+			)
+		)
+		(pin "1"
+		)
+		(pin "2"
+		)
+		(instances
+			(project "HPM5E31_ECatDualFOC"
+				(path "/a07e9810-3899-4327-ba8f-f24142a7c70e/0dcd211e-0cd3-4a5b-8381-64e2d1ceb9a5"
+					(reference "C152")
+					(unit 1)
+				)
+				(path "/a07e9810-3899-4327-ba8f-f24142a7c70e/395dcadf-6728-482a-9c72-95a7205ca2d1"
+					(reference "C153")
+					(unit 1)
+				)
