File: Hardware/SPI_Flash.kicad_sch (KiCad schematic)
At the start: 3 parts, among them U9 MX25L12833FM2I-10G

Commit message: 修存档拉线
Parts:
- renumbered C48 to C29, C49 to C30, U9 to U11
Changed lines of the file:
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@@
 		(on_board yes)
 		(dnp no)
-		(property "Reference" "C48"
+		(property "Reference" "C29"
 			(at 198.12 106.68 0)
 			(effects
@@
 		)
 		(pin "2"
+		)
+		(instances
+			(project "HPM5E31_ECatDualFOC"
+				(path "/a07e9810-3899-4327-ba8f-f24142a7c70e/39a16e10-36d8-4350-ab15-a79d4d0254e0"
+					(reference "C29")
+					(unit 1)
+				)
+			)
 		)
 	)
@@
 		(dnp no)
 		(fields_autoplaced yes)
-		(property "Reference" "U9"
+		(property "Reference" "U11"
 			(at 158.115 90.17 0)
 			(effects
@@
 		)
 		(pin "1"
+		)
+		(instances
+			(project "HPM5E31_ECatDualFOC"
+				(path "/a07e9810-3899-4327-ba8f-f24142a7c70e/39a16e10-36d8-4350-ab15-a79d4d0254e0"
+					(reference "U11")
+					(unit 1)
+				)
+			)
 		)
 	)
@@
 		(on_board yes)
 		(dnp no)
-		(property "Reference" "#PWR070"
+		(property "Reference" "#PWR085"
 			(at 207.01 101.6 0)
 			(effects
@@
 		)
 		(pin "1"
+		)
+		(instances
+			(project "HPM5E31_ECatDualFOC"
+				(path "/a07e9810-3899-4327-ba8f-f24142a7c70e/39a16e10-36d8-4350-ab15-a79d4d0254e0"
+					(reference "#PWR085")
+					(unit 1)
+				)
+			)
 		)
 	)
@@
 		(on_board yes)
 		(dnp no)
-		(property "Reference" "C49"
+		(property "Reference" "C30"
 			(at 205.74 104.14 0)
 			(effects
@@
 		)
 		(pin "2"
+		)
+		(instances
+			(project "HPM5E31_ECatDualFOC"
+				(path "/a07e9810-3899-4327-ba8f-f24142a7c70e/39a16e10-36d8-4350-ab15-a79d4d0254e0"
+					(reference "C30")
+					(unit 1)
+				)
+			)
 		)
 	)
@@
 		(dnp no)
 		(fields_autoplaced yes)
-		(property "Reference" "#PWR071"
+		(property "Reference" "#PWR087"
 			(at 207.01 114.3 0)
 			(effects
@@
 		)
 		(pin "1"
+		)
+		(instances
+			(project "HPM5E31_ECatDualFOC"
+				(path "/a07e9810-3899-4327-ba8f-f24142a7c70e/39a16e10-36d8-4350-ab15-a79d4d0254e0"
+					(reference "#PWR087")
+					(unit 1)
+				)
+			)
 		)
 	)
@@
 		(dnp no)
 		(fields_autoplaced yes)
-		(property "Reference" "#PWR072"
+		(property "Reference" "#PWR086"
 			(at 143.51 113.03 0)
 			(effects
@@
 		(pin "1"
 		)
-	)
+		(instances
+			(project "HPM5E31_ECatDualFOC"
+				(path "/a07e9810-3899-4327-ba8f-f24142a7c70e/39a16e10-36d8-4350-ab15-a79d4d0254e0"
+					(reference "#PWR086")
+					(unit 1)
+				)
+			)
+		)
+	)
