File: Hardware/HPM5E31_PINMAP_2.kicad_sch (KiCad schematic)
At the start: 15 parts, among them J21 WAFER-GH1.25-6PWB, J22 Conn_02x05_Odd_Even, U48 TXB0104RUTR, U49 TXS0108ERGYR

Commit message: 拉线
Connections:
- net EUI_CK: now also D32.4 (IO3), D32.7 (NC); no longer D32.1 (IO1), D32.10 (NC), J21.4 (Pin_4), U48.10 (B1)
- net EUI_DI: now also D32.1 (IO1), D32.10 (NC), J21.4 (Pin_4), U48.10 (B1); no longer D32.4 (IO3), D32.7 (NC), J21.2 (Pin_2), U48.8 (B3)
- net EUI_DO: now also D32.2 (IO2), D32.9 (NC), J21.3 (Pin_3), U48.9 (B2); no longer D32.5 (IO4), D32.6 (NC), J21.1 (Pin_1), U48.7 (B4)
- net EUI_SH: now also D32.5 (IO4), D32.6 (NC); no longer D32.2 (IO2), D32.9 (NC), J21.3 (Pin_3), U48.9 (B2)
- net PB26: now also U48.4 (A3); no longer U48.2 (A1)
- net PB27: now also U48.5 (A4); no longer U48.3 (A2)
- net PB28: now also U48.2 (A1); no longer U48.4 (A3)
- net PB29: now also U48.3 (A2); no longer U48.5 (A4)
- new net: J21.1 (Pin_1), U48.7 (B4)
- new net: J21.2 (Pin_2), U48.8 (B3)
Changed lines of the file:
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@@
-		)
-	)
-	(label "EUI_DO"
-		(at 214.63 76.2 180)
-		(effects
-			(font
-				(size 1.27 1.27)
-			)
-			(justify right bottom)
 		)
 	)
@@
 		)
 	)
-	(label "EUI_DI"
-		(at 214.63 73.66 180)
-		(effects
-			(font
-				(size 1.27 1.27)
-			)
-			(justify right bottom)
-		)
-	)
 	(label "ESC_GPIO_1"
 		(at 83.82 157.48 0)
@@
 		)
 	)
-	(label "EUI_CK"
-		(at 186.69 66.04 0)
-		(effects
-			(font
-				(size 1.27 1.27)
-			)
-			(justify left bottom)
-		)
-	)
 	(label "PD9"
 		(at 57.15 41.91 0)
@@
 		)
 	)
+	(label "PB26"
+		(at 181.61 44.45 0)
+		(effects
+			(font
+				(size 1.27 1.27)
+			)
+			(justify left bottom)
+		)
+	)
 	(label "ESC_GPIO_5"
 		(at 50.8 132.08 0)
@@
 		)
 	)
+	(label "EUI_DO"
+		(at 213.36 41.91 0)
+		(effects
+			(font
+				(size 1.27 1.27)
+			)
+			(justify left bottom)
+		)
+	)
 	(label "ESC_GPIO_0"
 		(at 83.82 104.14 0)
@@
 		)
 	)
+	(label "PB27"
+		(at 181.61 46.99 0)
+		(effects
+			(font
+				(size 1.27 1.27)
+			)
+			(justify left bottom)
+		)
+	)
 	(label "PC17"
 		(at 57.15 54.61 0)
@@
 		)
 	)
-	(label "EUI_DO"
-		(at 186.69 76.2 0)
-		(effects
-			(font
-				(size 1.27 1.27)
-			)
-			(justify left bottom)
-		)
-	)
 	(label "PB30"
 		(at 198.12 114.3 0)
@@
 		)
 	)
+	(label "EUI_DI"
+		(at 213.36 39.37 0)
+		(effects
+			(font
+				(size 1.27 1.27)
+			)
+			(justify left bottom)
+		)
+	)
+	(label "EUI_DO"
+		(at 186.69 68.58 0)
+		(effects
+			(font
+				(size 1.27 1.27)
+			)
+			(justify left bottom)
+		)
+	)
+	(label "EUI_DO"
+		(at 214.63 68.58 180)
+		(effects
+			(font
+				(size 1.27 1.27)
+			)
+			(justify right bottom)
+		)
+	)
 	(label "PD3"
 		(at 57.15 46.99 0)
@@
 		)
 	)
+	(label "EUI_SH"
+		(at 241.3 40.64 0)
+		(effects
+			(font
+				(size 1.27 1.27)
+			)
+			(justify left bottom)
+		)
+	)
 	(label "ESC_GPIO_4"
 		(at 52.07 157.48 0)
@@
 		)
 	)
-	(label "EUI_SH"
-		(at 186.69 68.58 0)
-		(effects
-			(font
-				(size 1.27 1.27)
-			)
-			(justify left bottom)
-		)
-	)
-	(label "PB28"
-		(at 181.61 44.45 0)
-		(effects
-			(font
-				(size 1.27 1.27)
-			)
-			(justify left bottom)
-		)
-	)
-	(label "EUI_SH"
-		(at 214.63 68.58 180)
-		(effects
-			(font
-				(size 1.27 1.27)
-			)
-			(justify right bottom)
-		)
-	)
-	(label "PB27"
-		(at 181.61 41.91 0)
-		(effects
-			(font
-				(size 1.27 1.27)
-			)
-			(justify left bottom)
-		)
-	)
-	(label "EUI_DI"
-		(at 186.69 73.66 0)
-		(effects
-			(font
-				(size 1.27 1.27)
-			)
-			(justify left bottom)
-		)
-	)
 	(label "ESC_GPIO_1"
 		(at 83.82 106.68 0)
@@
 		)
 	)
-	(label "EUI_SH"
-		(at 213.36 41.91 0)
-		(effects
-			(font
-				(size 1.27 1.27)
-			)
-			(justify left bottom)
+	(label "EUI_CK"
+		(at 214.63 73.66 180)
+		(effects
+			(font
+				(size 1.27 1.27)
+			)
+			(justify right bottom)
 		)
 	)
 	(label "EUI_DI"
-		(at 213.36 44.45 0)
-		(effects
-			(font
-				(size 1.27 1.27)
-			)
-			(justify left bottom)
-		)
-	)
-	(label "PB29"
-		(at 181.61 46.99 0)
-		(effects
-			(font
-				(size 1.27 1.27)
-			)
-			(justify left bottom)
-		)
-	)
-	(label "EUI_DO"
-		(at 213.36 46.99 0)
+		(at 186.69 66.04 0)
 		(effects
 			(font
@@
 		)
 	)
-	(label "PB26"
-		(at 181.61 39.37 0)
+	(label "EUI_CK"
+		(at 186.69 73.66 0)
 		(effects
 			(font
@@
 		)
 	)
-	(label "EUI_CK"
+	(label "EUI_DI"
 		(at 214.63 66.04 180)
+		(effects
+			(font
+				(size 1.27 1.27)
+			)
+			(justify right bottom)
+		)
+	)
+	(label "EUI_SH"
+		(at 186.69 76.2 0)
+		(effects
+			(font
+				(size 1.27 1.27)
+			)
+			(justify left bottom)
+		)
+	)
+	(label "PB29"
+		(at 181.61 41.91 0)
+		(effects
+			(font
+				(size 1.27 1.27)
+			)
+			(justify left bottom)
+		)
+	)
+	(label "EUI_SH"
+		(at 214.63 76.2 180)
 		(effects
 			(font
@@
 		)
 	)
-	(label "EUI_CK"
-		(at 213.36 39.37 0)
-		(effects
-			(font
-				(size 1.27 1.27)
-			)
-			(justify left bottom)
-		)
-	)
 	(label "ESC_GPIO_0"
 		(at 83.82 160.02 0)
@@
 		)
 	)
+	(label "PB28"
+		(at 181.61 39.37 0)
+		(effects
+			(font
+				(size 1.27 1.27)
+			)
+			(justify left bottom)
+		)
+	)
 	(label "ESC_GPIO_2"
 		(at 83.82 111.76 0)
@@
 		(effects
 			(font
+				(size 1.27 1.27)
+			)
+			(justify left bottom)
+		)
+	)
+	(label "EUI_CK"
+		(at 241.3 38.1 0)
+		(effects
+			(font

Commit message: 修存档拉线
Parts:
- renumbered C117 to C1, C124 to C2, C114 to C3, C116 to C4, D34 to D10, D32 to D6, D30 to D7, D33 to D8, D31 to D9, J21 to J5, J22 to J6, R114 to R12, R116 to R13, U49 to U1, U48 to U2

Commit message: 拉线
Connections:
- net EUI_CK: now also J5.2 (Pin_2), U2.8 (B3)
- net EUI_SH: now also J5.1 (Pin_1), U2.7 (B4)
Changed lines of the file:
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@@
 	)
 	(label "EUI_SH"
-		(at 241.3 40.64 0)
+		(at 213.36 46.99 0)
 		(effects
 			(font
@@
 	)
 	(label "EUI_CK"
-		(at 241.3 38.1 0)
-		(effects
-			(font
+		(at 213.36 44.45 0)
+		(effects
+			(font
