File: Hardware/HPM5E31_TOP.kicad_sch (KiCad schematic)
At the start: 17 parts, among them J1 Conn_Coaxial, J2 WAFER-ZH1.5-4PWB, J20 Conn_Coaxial, J3 Conn_02x05_Odd_Even, K1 DSHP02TSGET

Commit message: 新增ESC IO引出，ESC CTR LED，EUI接口
编码器接口电源输出加保险，SPI加ESD
PY32ADC外部接口加ESD
Parts:
- removed R1: 33R,1%, Resistor_SMD:R_0402_1005Metric, symbol HPM6280Foc:0402WGF330JTCE
- removed R4, R6: 4.7K,1%, Resistor_SMD:R_0402_1005Metric, symbol HPM6280Foc:0402WGF4701TCE
- added C114, C116: 100nF,16V, Capacitor_SMD:C_0402_1005Metric, symbol HPM6280Foc:CC0402KRX7R7BB104
- added D30, D31: RCLAMP3324P, Package_DFN_QFN:Diodes_UDFN-10_1.0x2.5mm_P0.5mm, symbol HPM6280Foc:RCLAMP3324P
- added D32: RCLAMP0524P, Package_DFN_QFN:Diodes_UDFN-10_1.0x2.5mm_P0.5mm, symbol HPM6280Foc:RCLAMP0524P
- added D33, D35: NCD0603G1, LED_SMD:LED_0603_1608Metric, symbol HPM6280Foc:NCD0603G1
- added D34, D36: NCD0603R1, LED_SMD:LED_0603_1608Metric, symbol HPM6280Foc:NCD0603R1
- added D37: NCD0603B1, LED_SMD:LED_0603_1608Metric, symbol HPM6280Foc:NCD0603B1
- added J21: WAFER-GH1.25-6PWB, Library:JST_GH_SM06B-GHS-TB_1x06-1MP_P1.25mm_Horizontal, symbol HPM6280Foc:WAFER-GH1.25-6PWB
- added J22: Conn_02x05_Odd_Even, Library:IDC_SMD_P1.27mm_02x05, symbol Connector_Generic:Conn_02x05_Odd_Even
- added R114, R116, R128, R129, R130: 2K,1%, Resistor_SMD:R_0402_1005Metric, symbol HPM6280Foc:0402WGF2001TCE
- added U48: TXB0104RUTR, Library:UQFN-12_1.7x2_Pitch0.4mm, symbol HPM6280Foc:TXB0104RUTR
Connections:
- net +3.3V: now also C114.1, R114.2, R116.2, R128.2, R129.2, R130.2, U48.1 (VCCA), U48.12 (OE)
- net GND: now also C114.2, C116.2, D30.3 (GND), D30.8 (NC), D31.3 (GND), D31.8 (NC), D32.3 (GND), D32.8 (NC), J21.6 (Pin_6), J21.MP (MountPin), J22.10 (Pin_10), J22.9 (Pin_9), U48.6 (GND)
- net PA0 renamed UART0.RXD
- net PA1 renamed UART0.TXD
- new net: D36.2 (A), R129.1
- new net: D35.2 (A), R128.1
- new net: D37.2 (A), R130.1
- new net: D33.2 (A), R114.1
- new net: D34.2 (A), R116.1
- new net +5V: C116.1, J21.1 (Pin_1), J22.1 (Pin_1), U48.11 (VCCB)
- new net ESC_CTR7: D33.1 (K)
- new net ESC_CTR8: D34.1 (K)
- new net EUI_CK: D32.1 (IO1), D32.10 (NC), J21.2 (Pin_2), U48.10 (B1)
- new net EUI_DI: D32.4 (IO3), D32.7 (NC), J21.4 (Pin_4), U48.8 (B3)
- new net EUI_DO: D32.5 (IO4), D32.6 (NC), J21.5 (Pin_5), U48.7 (B4)
- new net EUI_SH: D32.2 (IO2), D32.9 (NC), J21.3 (Pin_3), U48.9 (B2)
- new net PB26: U48.2 (A1)
- new net PB27: U48.3 (A2)
- new net PB28: U48.4 (A3)
- new net PB29: U48.5 (A4)
- new net PC18: D35.1 (K)
- new net PC19: D36.1 (K)
- new net PD1: D37.1 (K)
- new net PD10: D30.4 (IO3), D30.7 (NC), J22.7 (Pin_7)
- new net PD11: D31.1 (IO1), D31.10 (NC), J22.4 (Pin_4)
- new net PD12: D31.2 (IO2), D31.9 (NC), J22.6 (Pin_6)
- new net PD13: D31.4 (IO3), D31.7 (NC), J22.8 (Pin_8)
- new net PD4: D30.1 (IO1), D30.10 (NC), J22.3 (Pin_3)
- new net PD9: D30.2 (IO2), D30.9 (NC), J22.5 (Pin_5)
- no-connect marks 1 -> 6
Other:
- added sheet HPM5E31_PINMAP_1 (HPM5E31_PINMAP_1.kicad_sch)
- sheet HPM5E31_PORTA ports: added none; removed PA[0..31]
- sheet HPM5E31_PORTB ports: added none; removed PB[0..31]
- sheet HPM5E31_PORTC ports: added none; removed PC[0..31]
- sheet HPM5E31_PORTD ports: added none; removed PD[0..31]
- sheet HPM5E31_PORTE ports: added none; removed PE[0..5]
- sheet HPM5E31_PORTF ports: added none; removed PF[0..31]
- note added: "ESC_IO"
- note added: "ESC运行LED"
- note added: "ESC错误LED"
- note added: "EUI1"
- note added: "TRGM高速连接器"
- note added: "三色用户LED"
- note removed: "CAN0"
- note removed: "CAN3"
- note removed: "QEI0"
- note removed: "QEI1"
- note removed: "SPI1"
- note removed: "SPI2"
- note removed: "SPI3"
- note removed: "UART0"
- note removed: "UART4"
- note removed: "UART6"
- note removed: "UART7"
- moved on the sheet: J1, J20, R102, R103

Commit message: 调整引脚，拉线
Parts:
- removed C114, C116: 100nF,16V, Capacitor_SMD:C_0402_1005Metric, symbol HPM6280Foc:CC0402KRX7R7BB104
- removed D30, D31: RCLAMP3324P, Package_DFN_QFN:Diodes_UDFN-10_1.0x2.5mm_P0.5mm, symbol HPM6280Foc:RCLAMP3324P
- removed D32: RCLAMP0524P, Package_DFN_QFN:Diodes_UDFN-10_1.0x2.5mm_P0.5mm, symbol HPM6280Foc:RCLAMP0524P
- removed D33: NCD0603G1, LED_SMD:LED_0603_1608Metric, symbol HPM6280Foc:NCD0603G1
- removed D34: NCD0603R1, LED_SMD:LED_0603_1608Metric, symbol HPM6280Foc:NCD0603R1
- removed J21: WAFER-GH1.25-6PWB, Library:JST_GH_SM06B-GHS-TB_1x06-1MP_P1.25mm_Horizontal, symbol HPM6280Foc:WAFER-GH1.25-6PWB
- removed J22: Conn_02x05_Odd_Even, Library:IDC_SMD_P1.27mm_02x05, symbol Connector_Generic:Conn_02x05_Odd_Even
- removed R114, R116: 2K,1%, Resistor_SMD:R_0402_1005Metric, symbol HPM6280Foc:0402WGF2001TCE
- removed U48: TXB0104RUTR, Library:UQFN-12_1.7x2_Pitch0.4mm, symbol HPM6280Foc:TXB0104RUTR
- J1, J20: footprint Connector_Coaxial:MMCX_Molex_73415-1471_Vertical -> Connector_Coaxial:SMA_BAT_Wireless_BWSMA-KWE-Z001
Connections:
- net PC18 renamed PA20
- net PC19 renamed PA21
- net PD1 renamed PA22
- net UART0.RXD renamed PA0
- net UART0.TXD renamed PA1
- no-connect marks 6 -> 1
Other:
- added sheet HPM5E31_PINMAP_2 (HPM5E31_PINMAP_2.kicad_sch)
- note added: "UART0"
- note removed: "ESC_IO"
- note removed: "ESC运行LED"
- note removed: "ESC错误LED"
- note removed: "EUI1"

Commit message: 拉线
Parts:
- removed R102, R103: 33R,1%, Resistor_SMD:R_0402_1005Metric, symbol HPM6280Foc:0402WGF330JTCE
Connections:
- net PE4: now also J20.1 (In)
- net PE5: now also J1.1 (In)
- net PA20 renamed PC2
- net PA21 renamed PC3
- net PA22 renamed PC18

Commit message: 修存档拉线
Parts:
- renumbered D35 to D3, D36 to D4, D37 to D5, J20 to J1, J1 to J2, J2 to J3, J3 to J4, R2 to R1, R3 to R2, R5 to R3, R7 to R4, R8 to R5, R128 to R6, R129 to R7, R130 to R8

Commit message: 拉线
Parts:
- added R134: 10K,1%, Resistor_SMD:R_0402_1005Metric, symbol HPM6280Foc:0402WGF1002TCE
Connections:
- net +3.3V: now also R134.2
- net JTAG_TCK: now also D2.4 (IO3), D2.7 (NC); no longer D2.2 (IO2), D2.9 (NC)
- net JTAG_TDI: now also D2.5 (IO4), D2.6 (NC); no longer D1.5 (IO4), D1.6 (NC)
- net JTAG_TMS: now also D2.2 (IO2), D2.9 (NC); no longer D2.4 (IO3), D2.7 (NC)
- net JTAG_TRST: now also D1.5 (IO4), D1.6 (NC), R134.1; no longer D2.5 (IO4), D2.6 (NC)
- net PA0: now also D1.4 (IO3), D1.7 (NC); no longer D1.1 (IO1), D1.10 (NC)
- net PA1: now also D1.1 (IO1), D1.10 (NC); no longer D1.2 (IO2), D1.9 (NC)
- net ~{RESET}: now also D1.2 (IO2), D1.9 (NC); no longer D1.4 (IO3), D1.7 (NC)
Other:
- moved on the sheet: R3, R5

Commit message: 拉线
Changed lines of the file:
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@@
+	)
+	(bus_entry
+		(at 191.77 76.2)
+		(size -2.54 2.54)
+		(stroke
+			(width 0)
+			(type default)
+		)
 	)
 	(bus_entry
@@
 		)
 	)
+	(wire
+		(pts
+			(xy 177.8 78.74) (xy 189.23 78.74)
+		)
+		(stroke
+			(width 0)
+			(type default)
+		)
+	)
 	(bus
 		(pts
@@
 	(bus
 		(pts
-			(xy 191.77 72.39) (xy 191.77 86.36)
+			(xy 191.77 76.2) (xy 191.77 86.36)
 		)
 		(stroke
@@
 		(pts
 			(xy 205.74 110.49) (xy 203.2 110.49)
+		)
+		(stroke
+			(width 0)
+			(type default)
+		)
+	)
+	(bus
+		(pts
+			(xy 191.77 72.39) (xy 191.77 76.2)
 		)
 		(stroke
@@
 	(label "UART0.RXD"
 		(at 129.54 182.88 0)
+		(effects
+			(font
+				(size 1.27 1.27)
+			)
+			(justify left bottom)
+		)
+	)
+	(label "PE2"
+		(at 185.42 78.74 0)
 		(effects
 			(font
@@
 		(effects
 			(font
+				(size 1.27 1.27)
+			)
+			(justify right)
+		)
+	)
+	(hierarchical_label "BRAKE_RES_PWM"
+		(shape output)
+		(at 177.8 78.74 180)
+		(effects
+			(font

Commit message: 添加母线电压测量
Changed lines of the file:
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@@
+	)
+	(bus_entry
+		(at 158.75 151.13)
+		(size 2.54 -2.54)
+		(stroke
+			(width 0)
+			(type default)
+		)
 	)
 	(bus_entry
@@
 	)
 	(bus_entry
-		(at 154.94 148.59)
-		(size 2.54 -2.54)
-		(stroke
-			(width 0)
-			(type default)
-		)
-	)
-	(bus_entry
 		(at 154.94 187.96)
 		(size 2.54 -2.54)
@@
 	)
 	(bus_entry
+		(at 158.75 148.59)
+		(size 2.54 -2.54)
+		(stroke
+			(width 0)
+			(type default)
+		)
+	)
+	(bus_entry
 		(at 154.94 171.45)
 		(size 2.54 -2.54)
@@
 		)
 	)
+	(bus
+		(pts
+			(xy 161.29 146.05) (xy 161.29 148.59)
+		)
+		(stroke
+			(width 0)
+			(type default)
+		)
+	)
 	(wire
 		(pts
@@
 	(wire
 		(pts
+			(xy 140.97 151.13) (xy 158.75 151.13)
+		)
+		(stroke
+			(width 0)
+			(type default)
+		)
+	)
+	(wire
+		(pts
 			(xy 241.3 128.27) (xy 256.54 128.27)
 		)
@@
 		)
 	)
-	(bus
-		(pts
-			(xy 157.48 146.05) (xy 161.29 146.05)
-		)
-		(stroke
-			(width 0)
-			(type default)
-		)
-	)
 	(wire
 		(pts
@@
 	(wire
 		(pts
-			(xy 140.97 148.59) (xy 154.94 148.59)
+			(xy 140.97 148.59) (xy 158.75 148.59)
 		)
 		(stroke
@@
 	(label "PC2"
 		(at 36.83 168.91 0)
+		(effects
+			(font
+				(size 1.27 1.27)
+			)
+			(justify left bottom)
+		)
+	)
+	(label "PF27"
+		(at 149.86 151.13 0)
 		(effects
 			(font
@@
 		(effects
 			(font
+				(size 1.27 1.27)
+			)
+			(justify right)
+		)
+	)
+	(hierarchical_label "VBUS_ADC"
+		(shape input)
+		(at 140.97 151.13 180)
+		(effects
+			(font
